File: Eagle files/Main board - rev B/Lumiboard - main board (rev B).sch (EAGLE design)
At the start: 29 parts, among them IC1 MCP1700, IC2 ULN2003AD, U1 ATMEGA328, U2 DX_BT_MODULE, Y1 8Mhz

Commit message: New Eagle files
Parts:
- removed JP1: (no value), SparkFun:ARDUINO_SERIAL_PROGRAMLOCK
- removed JP6: M01PTH, SparkFun:M01PTH
- I2C: value (none) -> JP3
- JP7: value M01PTH -> FTDI; device SparkFun:M01PTH -> SparkFun:ARDUINO_SERIAL_PROGRAMLOCK
- LED1: value (none) -> JP5; device SparkFun:M03PTH -> SparkFun-Connectors:M04PTH
- LED2: value (none) -> JP6; device SparkFun:M03PTH -> SparkFun-Connectors:M04PTH
- POTSIN: value (none) -> JP4
- POTSPWR: value (none) -> JP2
- POWER: value (none) -> JP1
- renumbered POTS to POTSIN, PTS to POTSPWR
Connections:
- removed net N$17: IC2.O3, LED1.1
- removed net N$18: IC2.O2, LED1.2
- removed net N$19: IC2.O1, LED1.3
- new net N$14: IC2.O4, LED1.4
- new net N$15: IC2.O5, LED1.3
- new net N$16: IC2.O6, LED1.2
- net +5V: now also LED1.1, LED2.1; no longer JP6.1, JP7.1
- net 3.3V: now also JP7.VCC; no longer JP1.VCC
- net DTR: now also JP7.DTR; no longer JP1.DTR
- net GND: now also JP7.CTS, JP7.GND; no longer JP1.CTS, JP1.GND
- net N$1: now also IC2.O1, LED2.2; no longer IC2.O6, LED2.1
- net N$3: now also IC2.O2, LED2.3; no longer IC2.O5, LED2.2
- net N$5: now also IC2.O3, LED2.4; no longer IC2.O4, LED2.3
- net RXI: now also JP7.RXI, U1.PD1(TXD); no longer JP1.RXI, U1.PD0(RXD)
- net TXO: now also JP7.TXO, U1.PD0(RXD); no longer JP1.TXO, U1.PD1(TXD)

Commit message: New BOM, board files and readme
Parts:
- removed D3: DEBUG, led:LEDCHIPLED_0805
- removed I2C: JP3, SparkFun:M02PTH
- removed LED1: JP5, SparkFun-Connectors:M04PTH
- removed LED2: JP6, SparkFun-Connectors:M04PTH
- removed POTSIN: JP4, SparkFun:M03PTH
- removed POTSPWR: JP2, SparkFun:M02PTH
- removed POWER: JP1, SparkFun:M02PTH
- added H1, H2: STAND-OFFTIGHT, SparkFun:STAND-OFFTIGHT
- added J1: AVR_SPI_PRG_62X3_LOCK, SparkFun-Connectors:AVR_SPI_PRG_62X3_LOCK
- added J4: I2CDATA, SparkFun-Connectors:M022.54MM_SCREWTERM
- added JP1: POWER, SparkFun-Connectors:M022.54MM_SCREWTERM
- added JP10, JP11: (no value), SparkFun-Connectors:M03PTH
- added JP3: RGBLED2, SparkFun-Connectors:M04PTH
- added JP6: FTDI, SparkFun:ARDUINO_SERIAL_PROGRAMLOCK
- added JP8: POTSIN, SparkFun:M03PTH
- added JP9: POTPOWER, SparkFun:M02PTH
- added LOGO1: OSHW-LOGOL, SparkFun-Aesthetics:OSHW-LOGOL
- C2: value .1uF -> 1uF
- D1: value BLUE -> GREEN
- D2: value GREEN -> DEBUG
- JP2: value STAND-OFFTIGHT -> RGBLED1; device SparkFun:STAND-OFFTIGHT -> SparkFun-Connectors:M04PTH
- JP5: value STAND-OFFTIGHT -> 3V3OUT; device SparkFun:STAND-OFFTIGHT -> SparkFun-Connectors:M022.54MM_SCREWTERM
- JP7: value FTDI -> D4; device SparkFun:ARDUINO_SERIAL_PROGRAMLOCK -> SparkFun-Connectors:M01PTH
- SV1: value (none) -> SENSORS
- renumbered JP4 to H3
Connections:
- net N$11 renamed BTRESET
- removed net N$12: POTSIN.3, U1.PC2(ADC2)
- removed net N$14: IC2.O4, LED1.4
- removed net N$15: IC2.O5, LED1.3
- removed net N$16: IC2.O6, LED1.2
- removed net N$2: D1.A, U2.PIO8
- removed net N$20: POTSIN.2, U1.PC1(ADC1)
- removed net N$22: POTSIN.1, U1.PC0(ADC0)
- new net MISO: J1.1, U1.PB4(MISO)
- new net N$6: IC2.O5, JP2.3
- new net PD4: JP7.1, U1.PD4(XCK/T0)
- new net POT1: JP8.1, U1.PC0(ADC0)
- new net POT2: JP8.2, U1.PC1(ADC1)
- new net POT3: JP8.3, U1.PC2(ADC2)
- new net RESET: C2.2, J1.5, R4.1, U1.PC6(/RESET)
- new net SCK: J1.3, R2.2, U1.PB5(SCK)
- net +5V: now also JP1.2, JP2.1, JP3.1; no longer LED1.1, LED2.1, POWER.2
- net 3.3V: now also J1.2, JP5.2, JP6.VCC, JP9.2; no longer JP7.VCC, POTSPWR.2
- net B1: now also JP11.3
- net B2: now also JP10.3
- net BRX: now also U1.PD7(AIN1); no longer U1.PB4(MISO)
- net DTR: now also JP6.DTR; no longer JP7.DTR
- net G1: now also JP11.2
- net G2: now also JP10.2
- net GND: now also J1.6, JP1.1, JP5.1, JP6.CTS, JP6.GND, JP9.1; no longer D3.C, JP7.CTS, JP7.GND, POTSPWR.1, POWER.1
- net N$1: now also JP3.2; no longer LED2.2
- net N$10: now also IC2.O6, JP2.4; no longer C2.2, R4.1, U1.PC6(/RESET)
- net N$13: now also D2.A; no longer D3.A
- net N$3: now also JP3.3; no longer LED2.3
- net N$4: now also IC2.O4, JP2.2; no longer R2.2, U1.PB5(SCK)
- net N$5: now also JP3.4; no longer LED2.4
- net N$9: now also D1.A; no longer D2.A
- net R1: now also J1.4, JP11.1
- net R2: now also JP10.1
- net RXI: now also JP6.RXI; no longer JP7.RXI
- net SCL: now also J4.1; no longer I2C.1
- net SDA: now also J4.2; no longer I2C.2
- net TXO: now also JP6.TXO; no longer JP7.TXO
Other:
- note added: "ICSP header"
- moved on the sheet: C1, C2, C3, C4, D1, D2, IC1, IC2, R1, R2, R3, R4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
