File: Eagle files/Main board (rev C)/Lumiboard - main board (rev C).sch (EAGLE design)
At the start: 32 parts, among them IC1 MCP1700, IC2 ULN2003AD, J1 AVR_SPI_PRG_62X3_LOCK, J4 I2CDATA, U1 ATMEGA328, U2 DX_BT_MODULE, Y1 8Mhz

Commit message: Updated schematics and BOMs
Parts:
- removed J4: I2CDATA, SparkFun-Connectors:M022.54MM_SCREWTERM
- removed JP5: 3V3OUT, SparkFun-Connectors:M022.54MM_SCREWTERM
- removed JP7: D4, SparkFun-Connectors:M01PTH
- added C5, C6, C7: 0.1uF, SparkFun:CAP0805
- added JP4: I2C, SparkFun-Connectors:M04PTH
- C4: value 1uF -> 4.7uF
- IC1: value MCP1700 -> LM39300; device linear:MCP1703CB -> LM39300:LM39300
- LOGO1: value OSHW-LOGOL -> OSHW-LOGOS; device SparkFun-Aesthetics:OSHW-LOGOL -> SparkFun-Aesthetics:OSHW-LOGOS
- R1: value 82 -> 55; device resistor:R-US_R0805 -> SparkFun-Resistors:RESISTOR0805-RES
- R2, R3, R4: device resistor:R-US_R0805 -> SparkFun-Resistors:RESISTOR0805-RES
- Y1: value 8Mhz -> 8mHz
Connections:
- removed net PD4: JP7.1, U1.PD4(XCK/T0)
- net +5V: no longer R1.2
- net 3.3V: now also C5.2, C6.2, C7.2, JP4.4, R1.2; no longer JP5.2
- net GND: now also C5.1, C6.1, C7.1, JP4.3; no longer JP5.1
- net LIGHT: now also U1.ADC6; no longer U1.PC3(ADC3)
- net SCL: now also JP4.2; no longer J4.1
- net SDA: now also JP4.1; no longer J4.2
- net SOUND: now also U1.PC3(ADC3); no longer U1.ADC6
Other:
- moved on the sheet: C3, C4, IC1
