File: Eagle files/Sensor module (rev C)/Lumiboard - sensor module (rev C).brd (EAGLE design)
At the start: 42.9 x 16.3 mm, 16 parts, among them IC1 MCP9700SMD, M1 MIC9.7MM, Q2 TEMT6000, U1 OPA344

Commit message: Updated schematics and BOMs
Parts:
- moved C5 15.3 mm to (27.9, 11.9), turned to 270 degrees
- moved R4 5.36 mm to (22.1, 6.60), turned to 90 degrees
- moved R3 3.66 mm to (22.1, 9.91)
- moved C2 3.34 mm to (29.7, 11.9)
- moved R5 3.07 mm to (29.7, 8.64), turned to 90 degrees
- moved R2 2.34 mm to (26.2, 11.9), turned to 270 degrees
- moved C3 2.18 mm to (23.9, 6.60)
- moved C4 2.17 mm to (27.2, 4.83)
- moved R6 2.09 mm to (27.2, 6.35)
- moved IC1 1.52 mm to (16.0, 11.3)
- moved C1 1.02 mm to (13.3, 11.3)
- moved U1 0.51 mm to (26.7, 8.64)
- moved R1 0.40 mm to (12.7, 4.70), turned to 0 degrees
- moved Q2 0.25 mm to (17.0, 5.21)
Routing:
- net 3.3V: track 53.8 -> 42.5 mm, vias 2 -> 0
- net GND: track 0.00 -> 8.64 mm, vias 1 -> 6
- net N$1: track 6.43 -> 10.2 mm
- net N$7: track 8.23 -> 4.85 mm
- net TEMP: track 15.2 -> 12.5 mm
- net SOUND: track 39.5 -> 37.0 mm
- net LIGHT: track 12.8 -> 14.7 mm
- removed copper zone on layer 1, net GND
Other:
- board text added: "Rev C"
- board text removed: "Rev B"
